Commit message: Imported upstream version '0.1.5' of 'upstream'

File: turtlebot3_description/urdf/common_properties.xacro (robot description, xacro)
@@ -19,5 +19,5 @@
   </material>
   <material name="grey">
-    <color rgba="0.2 0.2 0.2 1.0"/>
+    <color rgba="0.5 0.5 0.5 1.0"/>
   </material>
   <material name="orange">

File: turtlebot3_description/urdf/turtlebot3_waffle.urdf.xacro (robot description, xacro)
@@ -29,5 +29,4 @@
         <box size="0.265 0.265 0.089"/>
       </geometry>
-      <material name="light_black"/>
     </collision>
     <inertial>
@@ -178,5 +177,5 @@
   </link>
   <joint name="camera_joint" type="fixed">
-    <origin xyz="0.076 -0.065 0.084" rpy="0 0 0"/>
+    <origin xyz="0.064 -0.065 0.094" rpy="0 0 0"/>
     <parent link="base_link"/>
     <child link="camera_link"/>
